File: kicad/lory.kicad_pcb (KiCad board)
At the start: 2 copper layers, 123.5 x 85.3 mm, 22 parts, among them J1 TRRS, SW10 SW_PUSH, SW11 SW_PUSH, SW12 SW_PUSH, SW14 SW_PUSH, SW15 SW_PUSH, SW16 SW_PUSH, SW17 SW_PUSH, SW18 SW_PUSH, SW2 SW_PUSH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

Commit message: Cleanup
Routing:
- net row2: track 124.2 -> 0.00 mm, vias 1 -> 0
- net SCL: track 113.7 -> 0.00 mm, vias 1 -> 0
- net col4: track 111.8 -> 0.00 mm
- net col5: track 97.9 -> 0.00 mm
- net col1: track 93.8 -> 0.00 mm
- net row1: track 92.6 -> 0.00 mm, vias 1 -> 0
- net Net-(U1-Pad12): track 85.0 -> 0.00 mm, vias 1 -> 0
- net GND: track 82.7 -> 0.00 mm
- net SDA: track 78.6 -> 0.00 mm, vias 1 -> 0
- net col3: track 76.7 -> 0.00 mm
- net row3: track 74.3 -> 0.00 mm, vias 1 -> 0
- net data: track 63.5 -> 0.00 mm
- net reset: track 61.5 -> 0.00 mm, vias 1 -> 0
- net row0: track 58.0 -> 0.00 mm, vias 1 -> 0
- net Net-(U1-Pad14): track 56.6 -> 0.00 mm
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- removed copper zone on B.Cu, net GND
- removed copper zone on F.Cu, net GND

Commit message: temp opean boardline
Parts:
- moved SW2 31.6 mm to (76.1, 104.6)
Other:
- board size 123.5 x 85.3 mm -> 130.6 x 85.3 mm
- net class Default removed
